File: output/pcbs/handlebar.kicad_pcb (KiCad board)
At the start: 2 copper layers, 155.2 x 111.6 mm, 17 parts

Commit message: update kicad files
Connections:
- MCU1 pad 1: (no net) -> net_index
- MCU1 pad 11: (no net) -> net_nums
- MCU1 pad 14: (no net) -> net_home
- MCU1 pad 15: (no net) -> net_top
- MCU1 pad 16: (no net) -> net_bottom
- MCU1 pad 2: (no net) -> net_middle
- MCU1 pad 5: (no net) -> net_ring
- MCU1 pad 7: (no net) -> net_inner
- S1 pad 1: B1 -> net_ring
- S10 pad 1: B3 -> net_index
- S11 pad 1: B3 -> net_index
- S12 pad 1: B3 -> net_index
- S13 pad 1: B4 -> net_inner
- S14 pad 1: B4 -> net_inner
- S15 pad 1: B4 -> net_inner
- S16 pad 1: B4 -> net_inner
- S2 pad 1: B1 -> net_ring
- S3 pad 1: B1 -> net_ring
- S4 pad 1: B1 -> net_ring
- S5 pad 1: B2 -> net_middle
- S6 pad 1: B2 -> net_middle
- S7 pad 1: B2 -> net_middle
- S8 pad 1: B2 -> net_middle
- S9 pad 1: B3 -> net_index
